Commit message: bittle

File: assets/descriptions/bittle/urdf/bittle.urdf (robot description, URDF)
Before this commit: robot bittle, 87 links, 86 joints
Links:
- link c_thlf_1: geometry collision mesh filename=c_thlf_1_collision.stl scale=0.001 0.001 0.001; visual mesh filename=c_thlf_1.stl scale=0.001 0.001 0.001
- link c_thlr_1: geometry collision mesh filename=c_thlr_1_collision.stl scale=0.001 0.001 0.001; visual mesh filename=c_thlr_1.stl scale=0.001 0.001 0.001
- link c_tholf_1: geometry collision mesh filename=c_tholf_1_collision.stl scale=0.001 0.001 0.001; visual mesh filename=c_tholf_1.stl scale=0.001 0.001 0.001
- link c_tholr__1: geometry collision mesh filename=c_tholr__1_collision.stl scale=0.001 0.001 0.001; visual mesh filename=c_tholr__1.stl scale=0.001 0.001 0.001
- link c_thorf_1: geometry collision mesh filename=c_thorf_1_collision.stl scale=0.001 0.001 0.001; visual mesh filename=c_thorf_1.stl scale=0.001 0.001 0.001
- link c_thorr_1: geometry collision mesh filename=c_thorr_1_collision.stl scale=0.001 0.001 0.001; visual mesh filename=c_thorr_1.stl scale=0.001 0.001 0.001
- link c_thrf__1: geometry collision mesh filename=c_thrf__1_collision.stl scale=0.001 0.001 0.001; visual mesh filename=c_thrf__1.stl scale=0.001 0.001 0.001
- link c_thrr_1: geometry collision mesh filename=c_thrr_1_collision.stl scale=0.001 0.001 0.001; visual mesh filename=c_thrr_1.stl scale=0.001 0.001 0.001
- link th_lf_1: geometry collision mesh filename=th_lf_1_collision.stl scale=0.001 0.001 0.001; visual mesh filename=th_lf_1.stl scale=0.001 0.001 0.001
- link th_lr__1: geometry collision mesh filename=th_lr__1_collision.stl scale=0.001 0.001 0.001; visual mesh filename=th_lr__1.stl scale=0.001 0.001 0.001
- link th_rf_1: geometry collision mesh filename=th_rf_1_collision.stl scale=0.001 0.001 0.001; visual mesh filename=th_rf_1.stl scale=0.001 0.001 0.001
- link th_rr_1: geometry collision mesh filename=th_rr_1_collision.stl scale=0.001 0.001 0.001; visual mesh filename=th_rr_1.stl scale=0.001 0.001 0.001
- link tho_lf_1: geometry collision mesh filename=tho_lf_1_collision.stl scale=0.001 0.001 0.001; visual mesh filename=tho_lf_1.stl scale=0.001 0.001 0.001
- link tho_lr_1: geometry collision mesh filename=tho_lr_1_collision.stl scale=0.001 0.001 0.001; visual mesh filename=tho_lr_1.stl scale=0.001 0.001 0.001
- link tho_rf__1: geometry collision mesh filename=tho_rf__1_collision.stl scale=0.001 0.001 0.001; visual mesh filename=tho_rf__1.stl scale=0.001 0.001 0.001
- link tho_rr_1: geometry collision mesh filename=tho_rr_1_collision.stl scale=0.001 0.001 0.001; visual mesh filename=tho_rr_1.stl scale=0.001 0.001 0.001
- link tube__1: geometry collision mesh filename=tube__1_collision.stl scale=0.001 0.001 0.001; visual mesh filename=tube__1.stl scale=0.001 0.001 0.001
- link tube_lf_1: geometry collision mesh filename=tube_lf_1_collision.stl scale=0.001 0.001 0.001; visual mesh filename=tube_lf_1.stl scale=0.001 0.001 0.001
- link tube_lr_1: geometry collision mesh filename=tube_lr_1_collision.stl scale=0.001 0.001 0.001; visual mesh filename=tube_lr_1.stl scale=0.001 0.001 0.001
- link tube_rr_1: geometry collision mesh filename=tube_rr_1_collision.stl scale=0.001 0.001 0.001; visual mesh filename=tube_rr_1.stl scale=0.001 0.001 0.001
